Commit message: [update] to utilize stereo_camera

File: wamv_description/urdf/sensors/stereo_camera/stereo_camera.urdf.xacro (robot description, xacro)
@@ -2,18 +2,18 @@
 <robot xmlns:xacro="http://ros.org/wiki/xacro" name="wam-v">
   <xacro:include filename="$(find wamv_description)/urdf/sensors/camera/camera.urdf.xacro"/>
-  <xacro:macro name="stereo_camera_v0" params="prefix parent base_line_length *origin">
+  <xacro:macro name="stereo_camera_v1" params="prefix parent base_line_length *origin">
     <!-- add link and joint -->
-    <link name="${prefix}_stereo_camera_base_link"/>
+    <link name="${prefix}_stereo_camera_link"/>
     <joint name="${prefix}_stereo_camera_joint" type="fixed">
       <insert_block name="origin"/>
       <parent link="${parent}"/>
-      <child link="${prefix}_stereo_camera_base_link"/>
+      <child link="${prefix}_stereo_camera_link"/>
     </joint>
     <!-- Left Camera -->
-    <xacro:camera_v0 prefix="left" parent="${prefix}_stereo_camera_base_link">
+    <xacro:camera_v0 prefix="${prefix}_stereo_left" parent="${prefix}_stereo_camera_link">
       <origin xyz="0 ${base_line_length*(0.5)} 0"/>
     </xacro:camera_v0>
     <!-- Right Camera -->
-    <xacro:camera_v0 prefix="right" parent="${prefix}_stereo_camera_base_link">
+    <xacro:camera_v0 prefix="${prefix}_stereo_right" parent="${prefix}_stereo_camera_link">
       <origin xyz="0 ${base_line_length*(-0.5)} 0"/>
     </xacro:camera_v0>
