Commit message: [update] to choose thruster position type

File: wamv_description/urdf/wamv_basic.urdf.xacro (robot description, xacro)
@@ -5,6 +5,22 @@
   <!-- Load engine macro -->
   <xacro:include filename="$(find wamv_description)/urdf/base/wamv_base.urdf.xacro"/>
-  <!-- Describe both engine -->
-  <xacro:engine prefix="left" position="-2.373776 1.027135 0.318237" />
-  <xacro:engine prefix="right" position="-2.373776 -1.027135 0.318237" />
+  <!-- Describe engine -->
+  <!-- Thruster Config -->
+  <xacro:arg name="thruster_config" default="H"/>
+  <xacro:property name="th_config" value="$(arg thruster_config)"/>
+  <xacro:if value="${th_config == 'H'}">
+    <xacro:engine prefix="left" position="-2.373776 1.027135 0.318237" />
+    <xacro:engine prefix="right" position="-2.373776 -1.027135 0.318237" />
+  </xacro:if>
+  <xacro:if value="${th_config == 'T'}">
+    <xacro:engine prefix="left" position="-2.373776 1.027135 0.318237" />
+    <xacro:engine prefix="right" position="-2.373776 -1.027135 0.318237" />
+    <xacro:engine prefix="lateral" position="0.0 0.0 0.318237" orientation="0.0 0.0 1.5707"/>
+  </xacro:if>
+  <xacro:if value="${th_config == 'X'}">
+    <xacro:engine prefix="left_rear" position="-2.373776 1.027135 0.318237"  orientation="0.0 0.0 0.785"/>
+    <xacro:engine prefix="right_rear" position="-2.373776 -1.027135 0.318237" orientation="0.0 0.0 -0.785"/>
+    <xacro:engine prefix="left_front" position="1.6 0.7  0.25" orientation="0.0 0.0 -0.785"/>
+    <xacro:engine prefix="right_front" position="1.6 -0.7 0.25" orientation="0.0 0.0 +0.785"/>
+  </xacro:if>
 </robot>

File: wamv_description/urdf/wamv_robotx.urdf.xacro (robot description, xacro)
@@ -1,6 +1,9 @@
 <?xml version="1.0"?>
 <robot xmlns:xacro="http://ros.org/wiki/xacro" name="WAM-V">
+  <xacro:arg name="thruster_config" default="H"/>
   <!-- Defines the basic WAM-V -->
-  <xacro:include filename="$(find wamv_description)/urdf/wamv_basic.urdf.xacro"/>
+  <xacro:include filename="$(find wamv_description)/urdf/wamv_basic.urdf.xacro">
+    <xacro:thruster_config value="$(arg thruster_config)"/>
+  </xacro:include>
   <!-- Defines Sensors -->
   <xacro:include filename="$(find wamv_description)/urdf/sensors/sensors.urdf.xacro"/>
