Commit message: [fix] typo

File: wamv_description/urdf/engine/engine.transmission.xacro (robot description, xacro)
@@ -4,6 +4,6 @@
     <transmission name="${prefix}_engine_transmission">
       <type>transmission_interface/SimpleTransmission</type>
-      <joint name="${prefix}_chasis_engine_jointt">
         <hardwareInterface>PositionJointInterface</hardwareInterface>
+      <joint name="${prefix}_chasis_engine_joint">
       </joint>
       <actuator name="${prefix}_engine_actuator">
