Commit message: [fix] to add base_footprint link

File: wamv_description/urdf/base/wamv_base.urdf.xacro (robot description, xacro)
@@ -81,4 +81,10 @@
     </collision>
   </xacro:macro>
+  <!-- base_footprint link -->
+  <link name="base_footprint"/>
+  <joint name="base_footprint_to_base_link" type="fixed">
+    <parent link="base_footprint"/>
+    <child link="base_link"/>
+  </joint>
   <!-- Basic model of the 16' WAM-V USV -->
   <link name="base_link">
