Commit message: [update] add ai pilot link
On here, you need to modify.

File: wamv_description/urdf/sensors/velodyne/velodyne.urdf.xacro (robot description, xacro)
@@ -15,4 +15,19 @@
       <origin xyz="1.5 0 0.8" rpy="0 0 0" />
     </xacro:VLP-16>
+    <!-- For adding AI Pilot model -->
+    <!-- 1. Comment out following part -->
+    <!-- 2. Write the path to ai pilot collada file -->
+    <!-- <link name="ai_pilot_link"> -->
+    <!--   <visual> -->
+	<!-- 	<geometry> -->
+	<!-- 	  <mesh filename="file://your_aipilot_dae path"/> -->
+	<!-- 	</geometry> -->
+	<!--   </visual> -->
+    <!-- </link> -->
+    <!-- <joint name="base_link_to_ai_pilot_link" type="fixed"> -->
+    <!--   <origin xyz="0.6 0 1.3"/> -->
+    <!--   <parent link="base_link"/> -->
+    <!--   <child link="ai_pilot_link"/> -->
+    <!-- </joint> -->
   </xacro:macro>
 </robot>
